File: the_skrillexinator/the_skrillexinator.kicad_sch (KiCad schematic)
At the start: 5 parts, among them J1 Conn_01x03, J2 Conn_01x03, U1 ESP32-WROOM-32

Commit message: add di pcb
Parts:
- J1, J2: footprint (none) -> Connector_PinHeader_2.54mm:PinHeader_1x03_P2.54mm_Vertical
Changed lines of the file:
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@@
 			)
 		)
-		(property "Footprint" ""
+		(property "Footprint" "Connector_PinHeader_2.54mm:PinHeader_1x03_P2.54mm_Vertical"
 			(at 186.69 78.74 0)
 			(hide yes)
@@
 			)
 		)
-		(property "Footprint" ""
+		(property "Footprint" "Connector_PinHeader_2.54mm:PinHeader_1x03_P2.54mm_Vertical"
 			(at 176.53 33.02 0)
 			(hide yes)
