File: the_skrillexinator/the_skrillexinator.kicad_pcb (KiCad board)
At the start: 2 copper layers, 3 parts, among them J1 Conn_01x03, J2 Conn_01x03, U1 ESP32-WROOM-32

Commit message: skibidi
Parts:
- moved J1 0.50 mm to (107.0, 91.7)
Changed lines of the file:
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@@
 	(footprint "Connector_PinHeader_2.54mm:PinHeader_1x03_P2.54mm_Vertical"
 		(layer "F.Cu")
-		(at 106.5 91.65)
+		(at 107 91.65)
 		(descr "Through hole straight pin header, 1x03, 2.54mm pitch, single row")
 		(tags "Through hole pin header THT 1x03 2.54mm single row")

Commit message: more pcbing
Parts:
- moved J1 43.0 mm to (147.0, 76.0)
- moved J2 16.4 mm to (121.5, 76.0)
Changed lines of the file:
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@@
 	(footprint "Connector_PinHeader_2.54mm:PinHeader_1x03_P2.54mm_Vertical"
 		(layer "F.Cu")
-		(at 116.61 91.65)
+		(at 121.5 76)
 		(descr "Through hole straight pin header, 1x03, 2.54mm pitch, single row")
 		(tags "Through hole pin header THT 1x03 2.54mm single row")
@@
 	(footprint "Connector_PinHeader_2.54mm:PinHeader_1x03_P2.54mm_Vertical"
 		(layer "F.Cu")
-		(at 107 91.65)
+		(at 147 76)
 		(descr "Through hole straight pin header, 1x03, 2.54mm pitch, single row")
 		(tags "Through hole pin header THT 1x03 2.54mm single row")

Commit message: wire that bi
Parts:
- moved J1 25.4 mm to (122.0, 71.5)
- moved J2 6.02 mm to (122.0, 82.0)
Routing:
- net GND: track 0.00 -> 49.2 mm
- net Net-(J1-Pin_1): track 0.00 -> 37.7 mm
- net Net-(J2-Pin_2): track 0.00 -> 23.2 mm
- net +3.3V: track 0.00 -> 20.8 mm

Commit message: help
Other:
- board outline added: 53.5 x 59.5 mm
Changed lines of the file:
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@@
 		)
+	)
+	(gr_rect
+		(start 107.012744 44.374673)
+		(end 160.555616 103.830627)
+		(stroke
+			(width 0.05)
+			(type default)
+		)
+		(fill no)
+		(layer "Edge.Cuts")
 	)
 	(segment

Commit message: HOORAHHHHH
Other:
- board size 53.5 x 59.5 mm -> 53.8 x 50.1 mm
Changed lines of the file:
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@@
 		(tags "Single 2.4 GHz Wi-Fi and Bluetooth combo  chip")
 		(property "Reference" "U1"
-			(at -10.61 8.43 90)
+			(at -0.5 2.43 90)
 			(layer "F.SilkS")
 			(effects
@@
 		(tags "Through hole pin header THT 1x03 2.54mm single row")
 		(property "Reference" "J2"
-			(at 0 -2.38 0)
+			(at -3 2.25 0)
 			(layer "F.SilkS")
 			(effects
@@
 		)
 		(property "Value" "Conn_01x03"
-			(at 0 7.46 0)
+			(at -6.75 0.5 0)
 			(layer "F.Fab")
 			(effects
@@
 		(tags "Through hole pin header THT 1x03 2.54mm single row")
 		(property "Reference" "J1"
-			(at 0 -2.38 0)
+			(at -2.75 2 0)
 			(layer "F.SilkS")
 			(effects
@@
 		)
 		(property "Value" "Conn_01x03"
-			(at 0 7.46 0)
+			(at -6.5 0.5 0)
 			(layer "F.Fab")
 			(effects
@@
 	(gr_rect
 		(start 107.012744 44.374673)
-		(end 160.555616 103.830627)
+		(end 160.786168 94.502682)
 		(stroke
 			(width 0.05)
@@
 	)
 	(segment
+		(start 129.26 85.31)
+		(end 143 85.31)
+		(width 0.2)
+		(layer "F.Cu")
+		(net "Net-(J2-Pin_2)")
+	)
+	(segment
+		(start 122 84.54)
+		(end 122 84.88)
+		(width 0.2)
+		(layer "F.Cu")
+		(net "Net-(J2-Pin_2)")
+	)
+	(segment
+		(start 124.45 87.33)
+		(end 127.24 87.33)
+		(width 0.2)
+		(layer "F.Cu")
+		(net "Net-(J2-Pin_2)")
+	)
+	(segment
+		(start 122 84.88)
+		(end 124.45 87.33)
+		(width 0.2)
+		(layer "F.Cu")
+		(net "Net-(J2-Pin_2)")
+	)
+	(segment
+		(start 127.24 87.33)
+		(end 129.26 85.31)
+		(width 0.2)
+		(layer "F.Cu")
+		(net "Net-(J2-Pin_2)")
+	)
+	(segment
 		(start 145.75 71.02)
 		(end 145.75 80)
@@
 		(net "Net-(J1-Pin_1)")
 	)
-	(segment
-		(start 129.26 85.31)
-		(end 143 85.31)
-		(width 0.2)
-		(layer "F.Cu")
-		(net "Net-(J2-Pin_2)")
-	)
-	(segment
-		(start 122 84.54)
-		(end 122 84.88)
-		(width 0.2)
-		(layer "F.Cu")
-		(net "Net-(J2-Pin_2)")
-	)
-	(segment
-		(start 124.45 87.33)
-		(end 127.24 87.33)
-		(width 0.2)
-		(layer "F.Cu")
-		(net "Net-(J2-Pin_2)")
-	)
-	(segment
-		(start 122 84.88)
-		(end 124.45 87.33)
-		(width 0.2)
-		(layer "F.Cu")
-		(net "Net-(J2-Pin_2)")
-	)
-	(segment
-		(start 127.24 87.33)
-		(end 129.26 85.31)
-		(width 0.2)
-		(layer "F.Cu")
-		(net "Net-(J2-Pin_2)")
-	)
 	(embedded_fonts no)
